File: hardware/board/clock_sync_16/clk_outputs_0_thru_7.kicad_sch (KiCad schematic)
At the start: 40 parts, among them J2 AudioJack3, U5 ISO6521FREUR

Commit message: route pcb v0.1
Parts:
- removed C10 (x14): 1uF, Capacitor_SMD:C_0402_1005Metric, symbol Device:C
- removed D1 (x7): D_TVS, Diode_SMD:D_0402_1005Metric, symbol Device:D_TVS
- removed J2 (x7): AudioJack3, Connector_Audio:Jack_3.5mm_CUI_SJ-3523-SMT_Horizontal, symbol Connector:AudioJack3
- removed U5 (x7): ISO6521FREUR, kicad_component_library:DFN-8_3x2mm_P0.5mm, symbol kicad_component_library:ISO6521FREUR
- added C10 (x14): 1uF, Capacitor_SMD:C_0402_1005Metric, symbol Device:C
- added D1 (x7): D_TVS, Diode_SMD:D_0402_1005Metric, symbol Device:D_TVS
- added D11, D12, D22, D26, D27, D28, D29, D8: LED, LED_SMD:LED_0603_1608Metric_Pad1.05x0.95mm_HandSolder, symbol Device:LED
- added J2 (x7): AudioJack3, kicad_component_library:Jack_3.5mm_Kycon_STX-3680-5NB_Vertical, symbol Connector:AudioJack3
- added R13, R14, R15, R16, R4, R5, R6, R7: R, Resistor_SMD:R_0402_1005Metric, symbol Device:R
- added U5 (x7): ISO6521FREUR, kicad_component_library:DFN-8_3x2mm_P0.5mm, symbol kicad_component_library:ISO6521FREUR
- J2: footprint Connector_Audio:Jack_3.5mm_CUI_SJ-3523-SMT_Horizontal -> kicad_component_library:Jack_3.5mm_Kycon_STX-3680-5NB_Vertical; Link https://www.digikey.com/en/products/detail/cui-devices/SJ-3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 -> https://www.digikey.com/en/products/detail/kycon-inc/STX-36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; Manufacturer (none) -> Kycon; Manufacturer Number SJ-3523-SMT-TR -> STX-3680-5NB; PCBWay Link https://www.pcbway.com/components/detail/SJ3523SMTTR/473228/ -> (none)
Connections:
- net +3.3V: now also C10.1, C10.1, C10.1, C10.1, C10.1, C10.1, C10.1, C10.1, U5.1 (VCC1), U5.1 (VCC1), U5.1 (VCC1), U5.1 (VCC1), U5.1 (VCC1), U5.1 (VCC1), U5.1 (VCC1)
- net CH1_CONNECTED: now also U5.2 (OUT)
- net CH2_CONNECTED: now also U5.2 (OUT)
- net CH3_CONNECTED: now also U5.2 (OUT)
- net CH4_CONNECTED: now also U5.2 (OUT)
- net CH5_CONNECTED: now also U5.2 (OUT)
- net CH6_CONNECTED: now also U5.2 (OUT)
- net CH7_CONNECTED: now also U5.2 (OUT)
- net GND: now also C10.2, C10.2, C10.2, C10.2, C10.2, C10.2, C10.2, U5.4 (GND1), U5.4 (GND1), U5.4 (GND1), U5.4 (GND1), U5.4 (GND1), U5.4 (GND1), U5.4 (GND1); no longer D1.1 (A1)
- net HARP_CLKOUT: now also U5.3 (INB), U5.3 (INB), U5.3 (INB), U5.3 (INB), U5.3 (INB), U5.3 (INB), U5.3 (INB)
- net at C10.1, J2.R, U5.7 (INA)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: now also R4.1
- net at C10.2, J2.S, U5.5 (GND2): now also D1.1 (A1), D22.1 (K)
- net at J2.T, U5.6 (OUTB): now also D1.2 (A2)
- removed net +3V3: C10.1, D1.2 (A2)
- new net: C10.1, J2.R, R13.1, U5.7 (INA), U5.8 (VCC2)
- new net: D26.2 (A), R13.2
- new net: C10.2, D1.1 (A1), D8.1 (K), J2.S, U5.5 (GND2)
- new net: D1.2 (A2), J2.T, U5.6 (OUTB) (x7)
- new net: C10.1, J2.R, R5.1, U5.7 (INA), U5.8 (VCC2)
- new net: C10.2, D1.1 (A1), D12.1 (K), J2.S, U5.5 (GND2)
- new net: D12.2 (A), R7.2
- new net: C10.1, J2.R, R15.1, U5.7 (INA), U5.8 (VCC2)
- new net: C10.2, D1.1 (A1), D28.1 (K), J2.S, U5.5 (GND2)
- new net: C10.1, J2.R, R14.1, U5.7 (INA), U5.8 (VCC2)
- new net: C10.2, D1.1 (A1), D27.1 (K), J2.S, U5.5 (GND2)
- new net: C10.1, J2.R, R16.1, U5.7 (INA), U5.8 (VCC2)
- new net: C10.2, D1.1 (A1), D29.1 (K), J2.S, U5.5 (GND2)
- new net: C10.1, J2.R, R7.1, U5.7 (INA), U5.8 (VCC2)
- new net: D29.2 (A), R16.2
- new net: D27.2 (A), R14.2
- new net: C10.1, J2.R, R6.1, U5.7 (INA), U5.8 (VCC2)
- new net: C10.2, D1.1 (A1), D11.1 (K), J2.S, U5.5 (GND2)
- new net: D22.2 (A), R4.2
- new net: D28.2 (A), R15.2
- new net: C10.2, D1.1 (A1), D26.1 (K), J2.S, U5.5 (GND2)
- new net: D8.2 (A), R5.2
- new net: D11.2 (A), R6.2
Other:
- note removed: "Harp Clk Sync ESD Protection. Near J1."
- note removed: "Harp Clock Sync Emitter (UART0)"
- moved on the sheet: C10, D1, J2, U5

Commit message: draft firmware
Parts:
- removed C10 (x16): 1uF, Capacitor_SMD:C_0402_1005Metric, symbol Device:C
- added C2 (x16): 100nF, Capacitor_SMD:C_0402_1005Metric, symbol Device:C
- R13, R14, R15, R16, R4, R5, R6, R7: value R -> 330; Link (none) -> https://www.digikey.com/en/products/detail/yageo/RC0402FR-0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
- U5: Manufacturer (none) -> Texas Instruments; Manufacturer Number (none) -> ISO6521FREUR
Connections:
- net +3.3V: now also C2.2, C2.2, C2.2, C2.2, C2.2, C2.2, C2.2, C2.2
- net GND: now also C2.1, C2.1, C2.1, C2.1, C2.1, C2.1, C2.1, C2.1
- net at J2.R, R13.1, U5.7 (INA)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: now also C2.1
- net at D1.1 (A1), D8.1 (K), J2.S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: now also C2.2
- net at J2.R, R5.1, U5.7 (INA)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: now also C2.1
- net at D1.1 (A1), D12.1 (K), J2.S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: now also C2.2
- net at J2.R, R15.1, U5.7 (INA)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: now also C2.1
- net at D1.1 (A1), D28.1 (K), J2.S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: now also C2.2
- net at J2.R, R14.1, U5.7 (INA)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: now also C2.1
- net at D1.1 (A1), D27.1 (K), J2.S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: now also C2.2
- net at J2.R, R16.1, U5.7 (INA)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: now also C2.1
- net at D1.1 (A1), D29.1 (K), J2.S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: now also C2.2
- net at J2.R, R7.1, U5.7 (INA)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: now also C2.1
- net at J2.R, R6.1, U5.7 (INA)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: now also C2.1
- net at D1.1 (A1), D11.1 (K), J2.S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: now also C2.2
- net at D1.1 (A1), D22.1 (K), J2.S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: now also C2.2
- net at D1.1 (A1), D26.1 (K), J2.S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: now also C2.2
- net at J2.R, R4.1, U5.7 (INA)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: now also C2.1

Commit message: dispatch works
Other:
- note added: "FIXME: R4 should be 1600KOhm to handle 3.3V & 5V options."
Changed lines of the file:
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@@
     (stroke (width 0) (type default))
+  )
+  (text "FIXME: R4 should\nbe 1600KOhm to\nhandle 3.3V & 5V\noptions."
+    (at 125.73 42.545 0)
+    (effects (font (size 2 2) (thickness 0.4) bold) (justify left bottom))
   )
   (global_label "HARP_CLKOUT" (shape input) (at 202.565 107.95 180) (fields_autoplaced)

Commit message: add pps/slow_uart output options
Parts:
- R13, R14, R15, R16, R4, R5, R6, R7: value 330 -> 1K6; Link https://www.digikey.com/en/products/detail/yageo/RC0402FR-0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 -> https://www.digikey.com/en/products/detail/panasonic-electr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; Manufacturer Number RC0402FR-07330RL -> ERJ-2RKF1601X
- renumbered C2 to C1, C2 to C24, C2 to C25, C2 to C26, C2 to C27, C2 to C28, C2 to C29, C2 to C3, C2 to C30, C2 to C31, C2 to C32, C2 to C33, C2 to C34, C2 to C35, C2 to C5, C2 to C7, D1 to D10, D1 to D13, D1 to D23, D1 to D24, D1 to D25, D1 to D6, D1 to D7, D1 to D9, J2 to J1, J2 to J10, J2 to J4, J2 to J5, J2 to J6, J2 to J7, J2 to J8, J2 to J9, U5 to U10, U5 to U11, U5 to U12, U5 to U6, U5 to U7, U5 to U8, U5 to U9
Other:
- note added: "1K6 Resistor handles 3.3V & 5V device currents."
- note removed: "FIXME: R4 should be 1600KOhm to handle 3.3V & 5V options."

Commit message: update harp core; update led resistors and deprecated parts; bump versions
Parts:
- D10, D13, D23, D24, D25, D6, D7, D9: Link https://www.digikey.com/en/products/detail/onsemi/ESD7571N2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 -> https://www.digikey.com/en/products/detail/nexperia-usa-inc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; Manufacturer Number ESD7571N2T5G -> PESD5V0F1BLD,315
Other:
- company: (none) -> The Allen Institute
- title: (none) -> harp.device.white-rabbit
Changed lines of the file:
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@@
 	(generator_version "8.0")
 	(paper "A4")
+	(title_block
+		(title "harp.device.white-rabbit")
+		(date "2025-02-21")
+		(rev "1.0.0")
+		(company "The Allen Institute")
+	)
 	(junction
 		(at 247.015 34.29)
@@
 			)
 		)
-		(property "Datasheet" "https://www.onsemi.com/pdf/datasheet/esd7571-d.pdf"
+		(property "Datasheet" "https://assets.nexperia.com/documents/data-sheet/PESD5V0F1BLD.pdf"
 			(at 104.775 151.13 0)
 			(effects
@@
 			)
 		)
-		(property "Link" "https://www.digikey.com/en/products/detail/onsemi/ESD7571N2T5G/7220690"
+		(property "Link" "https://www.digikey.com/en/products/detail/nexperia-usa-inc/PESD5V0F1BLD-315/3679473"
 			(at 104.775 151.13 0)
 			(effects
@@
 			)
 		)
-		(property "Manufacturer Number" "ESD7571N2T5G"
+		(property "Manufacturer Number" "PESD5V0F1BLD,315"
 			(at 104.775 151.13 0)
 			(effects
@@
 			)
 		)
-		(property "Datasheet" "https://www.onsemi.com/pdf/datasheet/esd7571-d.pdf"
+		(property "Datasheet" "https://assets.nexperia.com/documents/data-sheet/PESD5V0F1BLD.pdf"
 			(at 247.015 80.645 0)
 			(effects
@@
 			)
 		)
-		(property "Link" "https://www.digikey.com/en/products/detail/onsemi/ESD7571N2T5G/7220690"
+		(property "Link" "https://www.digikey.com/en/products/detail/nexperia-usa-inc/PESD5V0F1BLD-315/3679473"
 			(at 247.015 80.645 0)
 			(effects
@@
 			)
 		)
-		(property "Manufacturer Number" "ESD7571N2T5G"
+		(property "Manufacturer Number" "PESD5V0F1BLD,315"
 			(at 247.015 80.645 0)
 			(effects
@@
 			)
 		)
-		(property "Datasheet" "https://www.onsemi.com/pdf/datasheet/esd7571-d.pdf"
+		(property "Datasheet" "https://assets.nexperia.com/documents/data-sheet/PESD5V0F1BLD.pdf"
 			(at 104.775 44.45 0)
 			(effects
@@
 			)
 		)
-		(property "Link" "https://www.digikey.com/en/products/detail/onsemi/ESD7571N2T5G/7220690"
+		(property "Link" "https://www.digikey.com/en/products/detail/nexperia-usa-inc/PESD5V0F1BLD-315/3679473"
 			(at 104.775 44.45 0)
 			(effects
@@
 			)
 		)
-		(property "Manufacturer Number" "ESD7571N2T5G"
+		(property "Manufacturer Number" "PESD5V0F1BLD,315"
 			(at 104.775 44.45 0)
 			(effects
@@
 			)
 		)
-		(property "Datasheet" "https://www.onsemi.com/pdf/datasheet/esd7571-d.pdf"
+		(property "Datasheet" "https://assets.nexperia.com/documents/data-sheet/PESD5V0F1BLD.pdf"
 			(at 247.015 116.205 0)
 			(effects
@@
 			)
 		)
-		(property "Link" "https://www.digikey.com/en/products/detail/onsemi/ESD7571N2T5G/7220690"
+		(property "Link" "https://www.digikey.com/en/products/detail/nexperia-usa-inc/PESD5V0F1BLD-315/3679473"
 			(at 247.015 116.205 0)
 			(effects
@@
 			)
 		)
-		(property "Manufacturer Number" "ESD7571N2T5G"
+		(property "Manufacturer Number" "PESD5V0F1BLD,315"
 			(at 247.015 116.205 0)
 			(effects
@@
 			)
 		)
-		(property "Datasheet" "https://www.onsemi.com/pdf/datasheet/esd7571-d.pdf"
+		(property "Datasheet" "https://assets.nexperia.com/documents/data-sheet/PESD5V0F1BLD.pdf"
 			(at 104.775 115.57 0)
 			(effects
@@
 			)
 		)
-		(property "Link" "https://www.digikey.com/en/products/detail/onsemi/ESD7571N2T5G/7220690"
+		(property "Link" "https://www.digikey.com/en/products/detail/nexperia-usa-inc/PESD5V0F1BLD-315/3679473"
 			(at 104.775 115.57 0)
 			(effects
@@
 			)
 		)
-		(property "Manufacturer Number" "ESD7571N2T5G"
+		(property "Manufacturer Number" "PESD5V0F1BLD,315"
 			(at 104.775 115.57 0)
 			(effects
@@
 			)
 		)
-		(property "Datasheet" "https://www.onsemi.com/pdf/datasheet/esd7571-d.pdf"
+		(property "Datasheet" "https://assets.nexperia.com/documents/data-sheet/PESD5V0F1BLD.pdf"
 			(at 247.015 151.765 0)
 			(effects
@@
 			)
 		)
-		(property "Link" "https://www.digikey.com/en/products/detail/onsemi/ESD7571N2T5G/7220690"
+		(property "Link" "https://www.digikey.com/en/products/detail/nexperia-usa-inc/PESD5V0F1BLD-315/3679473"
 			(at 247.015 151.765 0)
 			(effects
@@
 			)
 		)
-		(property "Manufacturer Number" "ESD7571N2T5G"
+		(property "Manufacturer Number" "PESD5V0F1BLD,315"
 			(at 247.015 151.765 0)
 			(effects
@@
 			)
 		)
-		(property "Datasheet" "https://www.onsemi.com/pdf/datasheet/esd7571-d.pdf"
+		(property "Datasheet" "https://assets.nexperia.com/documents/data-sheet/PESD5V0F1BLD.pdf"
 			(at 104.775 80.01 0)
 			(effects
@@
 			)
 		)
-		(property "Link" "https://www.digikey.com/en/products/detail/onsemi/ESD7571N2T5G/7220690"
+		(property "Link" "https://www.digikey.com/en/products/detail/nexperia-usa-inc/PESD5V0F1BLD-315/3679473"
 			(at 104.775 80.01 0)
 			(effects
@@
 			)
 		)
-		(property "Manufacturer Number" "ESD7571N2T5G"
+		(property "Manufacturer Number" "PESD5V0F1BLD,315"
 			(at 104.775 80.01 0)
 			(effects
@@
 			)
 		)
-		(property "Datasheet" "https://www.onsemi.com/pdf/datasheet/esd7571-d.pdf"
+		(property "Datasheet" "https://assets.nexperia.com/documents/data-sheet/PESD5V0F1BLD.pdf"
 			(at 247.015 44.45 0)
 			(effects
@@
 			)
 		)
-		(property "Link" "https://www.digikey.com/en/products/detail/onsemi/ESD7571N2T5G/7220690"
+		(property "Link" "https://www.digikey.com/en/products/detail/nexperia-usa-inc/PESD5V0F1BLD-315/3679473"
 			(at 247.015 44.45 0)
 			(effects
@@
 			)
 		)
-		(property "Manufacturer Number" "ESD7571N2T5G"
+		(property "Manufacturer Number" "PESD5V0F1BLD,315"
 			(at 247.015 44.45 0)
 			(effects

Commit message: update missing BOM field
Parts:
- D10, D13, D23, D24, D25, D6, D7, D9: Manufacturer onsemi -> Nexperia USA Inc.
Changed lines of the file:
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@@
 			)
 		)
-		(property "Manufacturer" "onsemi"
+		(property "Manufacturer" "Nexperia USA Inc."
 			(at 104.775 151.13 0)
 			(effects
@@
 			)
 		)
-		(property "Manufacturer" "onsemi"
+		(property "Manufacturer" "Nexperia USA Inc."
 			(at 247.015 80.645 0)
 			(effects
@@
 			)
 		)
-		(property "Manufacturer" "onsemi"
+		(property "Manufacturer" "Nexperia USA Inc."
 			(at 104.775 44.45 0)
 			(effects
@@
 			)
 		)
-		(property "Manufacturer" "onsemi"
+		(property "Manufacturer" "Nexperia USA Inc."
 			(at 247.015 116.205 0)
 			(effects
@@
 			)
 		)
-		(property "Manufacturer" "onsemi"
+		(property "Manufacturer" "Nexperia USA Inc."
 			(at 104.775 115.57 0)
 			(effects
@@
 			)
 		)
-		(property "Manufacturer" "onsemi"
+		(property "Manufacturer" "Nexperia USA Inc."
 			(at 247.015 151.765 0)
 			(effects
@@
 			)
 		)
-		(property "Manufacturer" "onsemi"
+		(property "Manufacturer" "Nexperia USA Inc."
 			(at 104.775 80.01 0)
 			(effects
@@
 			)
 		)
-		(property "Manufacturer" "onsemi"
+		(property "Manufacturer" "Nexperia USA Inc."
 			(at 247.015 44.45 0)
 			(effects
