File: hardware/board/clock_sync_16/rp2040_with_usb.kicad_sch (KiCad schematic)
At the start: 43 parts, among them J2 AudioJack3, J3 USB_C_Receptacle_USB2.0, U1 TPD2EUSB30, U2 LP2985-3.3, U3 RP2040, U4 W25Q16JVUXIQ, X1 ECS-TXO-2016

Commit message: draft schematic
Parts:
- added J19: Conn_01x03_Male, Connector_PinHeader_2.54mm:PinHeader_1x03_P2.54mm_Vertical, symbol Connector:Conn_01x03_Male
Connections:
- net +3V3: no longer C23.2, U2.5 (VOUT), U3.1 (IOVDD), U3.10 (IOVDD), U3.22 (IOVDD), U3.26 (RUN), U3.33 (IOVDD), U3.42 (IOVDD), U3.43 (ADC_AVDD), U3.44 (VREG_IN), U3.48 (USB_VDD), U3.49 (IOVDD), X1.4 (VDD)
- net GND: now also J19.3 (Pin_3)
- net CH0_CONNECTED: now reaches U3.11 (GPIO8)
- net CH1_CONNECTED: now reaches U3.12 (GPIO9)
- net CH2_CONNECTED: now reaches U3.13 (GPIO10)
- net CH3_CONNECTED: now reaches U3.14 (GPIO11)
- net CH4_CONNECTED: now reaches U3.15 (GPIO12)
- net CH5_CONNECTED: now reaches U3.16 (GPIO13)
- net CH6_CONNECTED: now reaches U3.17 (GPIO14)
- net CH7_CONNECTED: now reaches U3.18 (GPIO15)
- net UART0_TXD: now reaches U3.2 (GPIO0)
- net UART0_TXD: now also J19.1 (Pin_1)
- net CH8_CONNECTED: now reaches U3.27 (GPIO16)
- net CH9_CONNECTED: now reaches U3.28 (GPIO17)
- net CH10_CONNECTED: now reaches U3.29 (GPIO18)
- net UART0_RXD: now reaches U3.3 (GPIO1)
- net UART0_RXD: now also J19.2 (Pin_2)
- net CH11_CONNECTED: now reaches U3.30 (GPIO19)
- net CH12_CONNECTED: now reaches U3.31 (GPIO20)
- net CH13_CONNECTED: now reaches U3.32 (GPIO21)
- net CH14_CONNECTED: now reaches U3.34 (GPIO22)
- net CH15_CONNECTED: now reaches U3.35 (GPIO23)
- net HARP_CLKOUT: now reaches U3.6 (GPIO4)
- net HARP_CLK_SYNC renamed HARP_CLKIN_SYNC
- new net +3.3V: C23.2, U2.5 (VOUT), U3.1 (IOVDD), U3.10 (IOVDD), U3.22 (IOVDD), U3.26 (RUN), U3.33 (IOVDD), U3.42 (IOVDD), U3.43 (ADC_AVDD), U3.44 (VREG_IN), U3.48 (USB_VDD), U3.49 (IOVDD), X1.4 (VDD)
- no-connect marks 35 -> 16
Other:
- note added: "(UART1TX) (UART1RX)"
- note added: "Debug Serial Port"
- note added: "TODO: "PPS CLKOUT" for Ephys"
- note removed: "(UART1RX)"
- note removed: "Note: Shield is connected to GND1 on PC side."
- moved on the sheet: C10, D1, D3, D4, J2, R1, R11, R12, SW2

Commit message: route pcb v0.1
Parts:
- added C52, C53: 1uF, Capacitor_SMD:C_0402_1005Metric, symbol Device:C
- added D22: LED, LED_SMD:LED_0603_1608Metric_Pad1.05x0.95mm_HandSolder, symbol Device:LED
- added D39: D_TVS, Diode_SMD:D_0402_1005Metric, symbol Device:D_TVS
- added J?: Conn_01x03_Female, Connector_Phoenix_MC:PhoenixContact_MCV_1,5_3-G-3.5_1x03_P3.50mm_Vertical, symbol Connector:Conn_01x03_Female
- added R4: R, Resistor_SMD:R_0402_1005Metric, symbol Device:R
- added U5: ISO6521FREUR, kicad_component_library:DFN-8_3x2mm_P0.5mm, symbol kicad_component_library:ISO6521FREUR
Connections:
- net +3V3 is gone; now on net +3.3V: C10.1, C11.1, C12.1, C13.2, C14.2, C15.2, C16.2, C17.2, C18.2, C19.2, C2.2, C20.2, C4.1, D1.2 (A2), J2.R, R8.2, U4.8 (VCC)
- net +3.3V: now also C52.1, U5.1 (VCC1)
- net CH0_CONNECTED: now also U3.27 (GPIO16); no longer U3.11 (GPIO8)
- net CH10_CONNECTED: now also U3.13 (GPIO10); no longer U3.29 (GPIO18)
- net CH11_CONNECTED: now also U3.14 (GPIO11); no longer U3.30 (GPIO19)
- net CH12_CONNECTED: now also U3.15 (GPIO12); no longer U3.31 (GPIO20)
- net CH13_CONNECTED: now also U3.16 (GPIO13); no longer U3.32 (GPIO21)
- net CH14_CONNECTED: now also U3.17 (GPIO14); no longer U3.34 (GPIO22)
- net CH15_CONNECTED: now also U3.18 (GPIO15); no longer U3.35 (GPIO23)
- net CH1_CONNECTED: now also U3.28 (GPIO17); no longer U3.12 (GPIO9)
- net CH2_CONNECTED: now also U3.29 (GPIO18); no longer U3.13 (GPIO10)
- net CH3_CONNECTED: now also U3.30 (GPIO19); no longer U3.14 (GPIO11)
- net CH4_CONNECTED: now also U3.31 (GPIO20); no longer U3.15 (GPIO12)
- net CH5_CONNECTED: now also U3.32 (GPIO21); no longer U3.16 (GPIO13)
- net CH6_CONNECTED: now also U3.34 (GPIO22); no longer U3.17 (GPIO14)
- net CH7_CONNECTED: now also U3.35 (GPIO23); no longer U3.18 (GPIO15)
- net CH8_CONNECTED: now also U3.11 (GPIO8); no longer U3.27 (GPIO16)
- net CH9_CONNECTED: now also U3.12 (GPIO9); no longer U3.28 (GPIO17)
- net GND: now also C52.2, U5.4 (GND1)
- net SLOW_CLKOUT_CONNECTED: now reaches U3.4 (GPIO2)
- net SLOW_CLKOUT_CONNECTED: now also U5.2 (OUT)
- net UART0_TXD renamed SLOW_CLKOUT
- net SLOW_CLKOUT: now also U5.3 (INB)
- new net: C53.2, D22.1 (K), D39.1 (A1), J?.3 (Pin_3), U5.5 (GND2)
- new net: D39.2 (A2), J?.1 (Pin_1), U5.6 (OUTB)
- new net: C53.1, J?.2 (Pin_2), R4.1, U5.7 (INA), U5.8 (VCC2)
- new net: D22.2 (A), R4.2
- no-connect marks 16 -> 15
Other:
- note added: ""Debug Serial Port" and "Slow Harp Clock Emitter" share UART0."
- note added: "(UART0_TXD)"
- note added: "C11 must be near VREG_IN."
- note added: "Slow Harp Clock Emitter"
- note removed: "C10 must be near VREG_IN."
- note removed: "RP2040 VREG_IN Bypass Cap"
- note removed: "TODO: "PPS CLKOUT" for Ephys"
- moved on the sheet: C10, C11, C2, C4, D1, D2, D3, D4, FID1, FID2, FID3, J19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

Commit message: draft v0.1 pcb
Parts:
- removed U2: LP2985-3.3, Package_TO_SOT_SMD:SOT-23-5, symbol Regulator_Linear:LP2985-3.3
- added U2: TPS73433DDCR, Package_TO_SOT_SMD:SOT-23-5, symbol kicad_component_library:TPS73433DDCR
Connections:
- net +3.3V: now also U2.5 (OUT)
- net GND: now also U2.2 (GND)
- net VDD: now also U2.1 (IN), U2.3 (EN)
- net at C21.1: now also U2.4 (NR)

Commit message: draft firmware
Parts:
- C52, C53: value 1uF -> 100nF; Link https://www.digikey.com/en/products/detail/murata-electroni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 -> https://www.digikey.com/en/products/detail/walsin-technolog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; Manufacturer Murata Electronics -> Walson Technology Corporation; Manufacturer Number GRM155R6YA105KE11J -> 0402B104K160CT; Notes must not be polarized -> (none); PCBWay Link (none) -> https://www.pcbway.com/components/detail/0402B104K160CT/307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; Rated Voltage 35V -> 16V; Temperature Coefficient X5R -> X7R; Tolerance (none) -> 10%
- J2: Manufacturer (none) -> CUI Devices
- J?: Notes Mates with 1863165, 1862865 -> Mates with 1862865
- R11, R12: Link https://www.digikey.com/en/products/detail/panasonic-electr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 -> https://www.digikey.com/en/products/detail/yageo/RC0402FR-0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; Manufacturer Panasonic Electronic Components -> Yageo; Manufacturer Number ERA-2AEB331X -> RC0402FR-07330RL
- R4: value R -> 330; Link (none) -> https://www.digikey.com/en/products/detail/yageo/RC0402FR-0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
- U2: Link (none) -> https://www.digikey.com/en/products/detail/texas-instrument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; Manufacturer (none) -> Texas Instruments; Manufacturer Number (none) -> TPS73433DDCR
- U5: Manufacturer (none) -> Texas Instruments; Manufacturer Number (none) -> ISO6521FREUR
Connections:
- net +3.3V: now also C52.2; no longer C52.1
- net GND: now also C52.1; no longer C52.2
- net at D22.1 (K), D39.1 (A1), J?.3 (Pin_3)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: now also C53.1; no longer C53.2
- net at J?.2 (Pin_2), R4.1, U5.7 (INA)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: now also C53.2; no longer C53.1

Commit message: add pps/slow_uart output options
Parts:
- J2: footprint Connector_Audio:Jack_3.5mm_CUI_SJ-3523-SMT_Horizontal -> Connector_Audio:Jack_3.5mm_CUI_SJ-3524-SMT_Horizontal; Alternate (none) -> SJ-3523-SMT-TR; Manufacturer Number SJ-3523-SMT-TR -> SJ-3524-SMT-TR; PCBWay Link https://www.pcbway.com/components/detail/SJ3523SMTTR/473228/ -> (none)
- R11, R12: Notes (none) -> indicator LED
- R25: renamed from R4; value 330 -> 1K6; Link https://www.digikey.com/en/products/detail/yageo/RC0402FR-0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 -> https://www.digikey.com/en/products/detail/panasonic-electr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; Manufacturer Number RC0402FR-07330RL -> ERJ-2RKF1601X
- renumbered D22 to D38, U5 to U22

Commit message: update harp core; update led resistors and deprecated parts; bump versions
Parts:
- D1, D2, D39: Link https://www.digikey.com/en/products/detail/onsemi/ESD7571N2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 -> https://www.digikey.com/en/products/detail/nexperia-usa-inc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; Manufacturer Number ESD7571N2T5G -> PESD5V0F1BLD,315
Other:
- title: (none) -> harp.device.white-rabbit
Changed lines of the file:
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@@
 	(paper "A4")
 	(title_block
-		(rev "0.1")
+		(title "harp.device.white-rabbit")
+		(date "2025-02-21")
+		(rev "1.0.0")
 		(company "The Allen Institute")
 	)
@@
 			)
 		)
-		(property "Datasheet" "https://www.onsemi.com/pdf/datasheet/esd7571-d.pdf"
+		(property "Datasheet" "https://assets.nexperia.com/documents/data-sheet/PESD5V0F1BLD.pdf"
 			(at 74.93 155.575 0)
 			(effects
@@
 			)
 		)
-		(property "Link" "https://www.digikey.com/en/products/detail/onsemi/ESD7571N2T5G/7220690"
+		(property "Link" "https://www.digikey.com/en/products/detail/nexperia-usa-inc/PESD5V0F1BLD-315/3679473"
 			(at 74.93 155.575 0)
 			(effects
@@
 			)
 		)
-		(property "Manufacturer Number" "ESD7571N2T5G"
+		(property "Manufacturer Number" "PESD5V0F1BLD,315"
 			(at 74.93 155.575 0)
 			(effects
@@
 			)
 		)
-		(property "Datasheet" "https://www.onsemi.com/pdf/datasheet/esd7571-d.pdf"
+		(property "Datasheet" "https://assets.nexperia.com/documents/data-sheet/PESD5V0F1BLD.pdf"
 			(at 28.575 99.06 0)
 			(effects
@@
 			)
 		)
-		(property "Link" "https://www.digikey.com/en/products/detail/onsemi/ESD7571N2T5G/7220690"
+		(property "Link" "https://www.digikey.com/en/products/detail/nexperia-usa-inc/PESD5V0F1BLD-315/3679473"
 			(at 28.575 99.06 0)
 			(effects
@@
 			)
 		)
-		(property "Manufacturer Number" "ESD7571N2T5G"
+		(property "Manufacturer Number" "PESD5V0F1BLD,315"
 			(at 28.575 99.06 0)
 			(effects
@@
 			)
 		)
-		(property "Datasheet" "https://www.onsemi.com/pdf/datasheet/esd7571-d.pdf"
+		(property "Datasheet" "https://assets.nexperia.com/documents/data-sheet/PESD5V0F1BLD.pdf"
 			(at 82.55 59.055 0)
 			(effects
@@
 			)
 		)
-		(property "Link" "https://www.digikey.com/en/products/detail/onsemi/ESD7571N2T5G/7220690"
+		(property "Link" "https://www.digikey.com/en/products/detail/nexperia-usa-inc/PESD5V0F1BLD-315/3679473"
 			(at 82.55 59.055 0)
 			(effects
@@
 			)
 		)
-		(property "Manufacturer Number" "ESD7571N2T5G"
+		(property "Manufacturer Number" "PESD5V0F1BLD,315"
 			(at 82.55 59.055 0)
 			(effects

Commit message: update missing BOM field
Parts:
- D1, D2, D39: Manufacturer onsemi -> Nexperia USA Inc.
Changed lines of the file:
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@@
 			)
 		)
-		(property "Manufacturer" "onsemi"
+		(property "Manufacturer" "Nexperia USA Inc."
 			(at 74.93 155.575 0)
 			(effects
@@
 			)
 		)
-		(property "Manufacturer" "onsemi"
+		(property "Manufacturer" "Nexperia USA Inc."
 			(at 28.575 99.06 0)
 			(effects
@@
 			)
 		)
-		(property "Manufacturer" "onsemi"
+		(property "Manufacturer" "Nexperia USA Inc."
 			(at 82.55 59.055 0)
 			(effects
